Commit message: Worked on Fine Tuning 1

File: description/robot_core.xacro (robot description, xacro)
@@ -19,4 +19,12 @@
     <!-- BASE LINK -->
     <link name="base_link">
+    </link>
+    <!-- BASE FOOTPRINT -->
+    <joint name="base_footprint_joint" type="fixed">
+        <parent link="base_link"/>
+        <child link="base_footprint"/>
+        <origin xyz="0 0 0" rpy="0 0 0"/>
+    </joint>
+    <link name="base_footprint">
     </link>
     <joint name="chassis_joint" type="fixed">

File: description/ros2_control.xacro (robot description, xacro)
@@ -11,5 +11,5 @@
                 <param name="baud_rate">57600</param>
                 <param name="timeout">1000</param>
-                <param name="enc_counts_per_rev">12532</param>
+                <param name="enc_counts_per_rev">20000</param>
             </hardware>
             <joint name="left_wheel_joint">

Commit message: Check

File: description/robot_core.xacro (robot description, xacro)
@@ -36,5 +36,5 @@
     <link name="chassis">
         <visual>
-        	<origin xyz="0.165 0 0.075"/>
+        <origin xyz="0.165 0 0.075"/>
             <geometry>
                 <box size="0.33 0.25 0.15"/>

File: description/ros2_control.xacro (robot description, xacro)
@@ -11,5 +11,5 @@
                 <param name="baud_rate">57600</param>
                 <param name="timeout">1000</param>
-                <param name="enc_counts_per_rev">20000</param>
+                <param name="enc_counts_per_rev">11000</param>
             </hardware>
             <joint name="left_wheel_joint">
